File: picoKey_2304.brd (EAGLE design)
At the start: 78 x 125 mm, 76 parts, among them U1 CHG-4056

Commit message: 80
Parts:
- removed U$1: FEATHER_WING_OLED, picoKey:FEATHER_WING_OLED
- added TP1, TP2, TP3, TP4: TPTP06R, testpad:TP06R
- added U2: FEATHER_WING_OLED, picoKey:FEATHER_WING_OLED
- D1, D10, D11, D12, D13, D14, D15, D16, D17, D18, D19, D2, D20, D3, D4, D5, D6, D7, D8, D9: value 1N4148WS -> 1N4148WS123; device SamacSys_Parts:SODFL2512X90N -> SamacSys_Parts:SOD-123
- D21: value (none) -> 1N4148WS
- moved LED16 58.0 mm to (68.5, 35.2)
- moved LED8 58.0 mm to (68.5, 73.2)
- moved LED13 56.0 mm to (11.5, 35.2)
- moved LED5 56.0 mm to (11.5, 73.2)
- moved LED0 29.8 mm to (72.0, 103.6), turned to 270 degrees
- moved R9 24.4 mm to (68.0, 103.6), turned to 0 degrees
- moved R6 21.3 mm to (48.5, 123.1)
- moved LED15 20.1 mm to (49.5, 35.2)
- moved LED7 20.1 mm to (49.5, 73.2)
- moved R5 19.6 mm to (51.0, 123.1)
- moved LED14 18.1 mm to (30.5, 35.2)
- moved LED6 18.1 mm to (30.5, 73.2)
- moved D8 15.5 mm to (61.0, 24.6)
- moved D2 15.0 mm to (23.0, 5.60)
- moved D3 15.0 mm to (42.0, 5.60)
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Connections:
- net N$29 renamed 4.2V
- removed net N$26: U$1.13
- removed net N$41: X1.GP10
- net 3V3: now also U2.15; no longer U$1.15
- net A_BTN: now also U2.26; no longer U$1.26
- net B_BTN: now also U2.25; no longer U$1.25
- net C_BTN: now also U2.24, X1.GP6; no longer U$1.24
- net GND: now also U2.13
- net N$10: now also D6.A; no longer D6.2
- net N$11: now also D7.A; no longer D7.2
- net N$12: now also D8.A; no longer D8.2
- net N$13: now also D9.A; no longer D9.2
- net N$14: now also D10.A; no longer D10.2
- net N$15: now also D11.A; no longer D11.2
- net N$16: now also D12.A; no longer D12.2
- net N$17: now also D13.A; no longer D13.2
- net N$18: now also D14.A; no longer D14.2
- net N$19: now also D15.A; no longer D15.2
- net N$20: now also D16.A; no longer D16.2
- net N$21: now also D17.A; no longer D17.2
- net N$22: now also D18.A; no longer D18.2
- net N$24: now also D20.A; no longer D20.2
- net N$25: now also D19.A; no longer D19.2
- net N$38: now also TP1.TP
- net N$40: now also TP2.TP
- net N$5: now also D1.A; no longer D1.2
- net N$6: now also D2.A; no longer D2.2
- net N$7: now also D3.A; no longer D3.2
- net N$8: now also D4.A; no longer D4.2
- net N$9: now also D5.A; no longer D5.2
- net ROW1: now also D1.K, D2.K, D3.K, D4.K; no longer D1.1, D2.1, D3.1, D4.1
- net ROW2: now also D5.K, D6.K, D7.K, D8.K; no longer D5.1, D6.1, D7.1, D8.1
- net ROW3: now also D10.K, D11.K, D12.K, D9.K; no longer D10.1, D11.1, D12.1, D9.1
- net ROW4: now also D13.K, D14.K, D15.K, D16.K; no longer D13.1, D14.1, D15.1, D16.1
- net ROW5: now also D17.K, D18.K, D19.K, D20.K; no longer D17.1, D18.1, D19.1, D20.1
- net RX: now also TP4.TP
- net SCL: now also U2.27; no longer U$1.27
- net SDA: now also U2.28; no longer U$1.28
- net TX: now also TP3.TP
Routing:
- net VSYS: track 0.00 -> 614.1 mm, vias 0 -> 31
- net COL1: track 0.00 -> 141.4 mm
- net COL4: track 0.00 -> 134.7 mm, vias 0 -> 1
- net COL3: track 0.00 -> 123.0 mm, vias 0 -> 1
- net COL2: track 0.00 -> 121.4 mm
- net ROW1: track 0.00 -> 116.0 mm, vias 0 -> 1
- net ROW2: track 0.00 -> 100.8 mm, vias 0 -> 1
- net LED13: track 0.00 -> 93.9 mm
- net LED5: track 0.00 -> 93.0 mm
- net LED9: track 0.00 -> 92.5 mm
- net LED17: track 0.00 -> 92.2 mm
- net ROW3: track 0.00 -> 86.6 mm, vias 0 -> 1
- net ROW4: track 0.00 -> 73.0 mm, vias 0 -> 2
- net C_BTN: track 0.00 -> 63.7 mm
- net 3V3: track 0.00 -> 63.3 mm
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- added copper zone on layer 1, net 4.2V
- added copper zone on layer 1, net GND
- added copper zone on layer 16, net GND
- added copper zone on layer 1, net VSYS
- removed copper zone on layer 1, net N$28
- removed copper zone on layer 16, net N$28
Other:
- board size 78 x 125 mm -> 80 x 126 mm
- board text added: "エンター スタビライザー"
