File: picoKey_2304.brd (EAGLE design)
At the start: 80 x 126 mm, 78 parts, among them U1 CHG-4056, U2 FEATHER_WING_OLED

Commit message: fix
Routing:
- net VSYS: track 589.5 -> 563.0 mm, vias 31 -> 29
- net LED17: track 100.3 -> 99.7 mm
- net 3V3: track 63.3 -> 63.8 mm
