File: picoKey_2304.sch (EAGLE design)
At the start: 76 parts, among them U1 CHG-4056

Commit message: 80
Parts:
- added TP1, TP2, TP3, TP4: TPTP06R, testpad:TPTP06R
- D1, D10, D11, D12, D13, D14, D15, D16, D17, D18, D19, D2, D20, D3, D4, D5, D6, D7, D8, D9: value 1N4148WS -> 1N4148WS123; device SamacSys_Parts:1N4148WS -> SamacSys_Parts:1N4148WS123
- D21: value (none) -> 1N4148WS
- renumbered U$1 to U2
Connections:
- net N$29 renamed 4.2V
- removed net N$26: U2.GND@1
- removed net N$41: X1.GP10
- net C_BTN: now also X1.GP6
- net GND: now also U2.GND@1
- net N$38: now also TP1.TP
- net N$40: now also TP2.TP
- net RX: now also TP4.TP
- net TX: now also TP3.TP
