File: picoKey_230407-e.brd (EAGLE design)
At the start: 80 x 126 mm, 78 parts, among them U1 CHG-4056, U2 FEATHER_WING_OLED

Commit message: edit enter
Parts:
- moved D8 13.5 mm to (74.4, 13.5), turned to 0 degrees
- moved S8 8.34 mm to (74.4, 21.0), turned to 90 degrees
- moved LED16 6.65 mm to (63.8, 21.0), turned to 90 degrees
- moved TP1 2.24 mm to (59.0, 19.6)
Routing:
- net LED17: track 100.3 -> 62.0 mm, vias 0 -> 2
- net ROW2: track 108.5 -> 124.9 mm
- net LED16: track 20.9 -> 33.3 mm
- net COL4: track 113.7 -> 106.5 mm
- net VSYS: track 589.5 -> 582.3 mm
- net LED20: track 5.28 -> 7.70 mm
Other:
- board text added: "エンター スタビライザー"
