File: picoKey_230407.brd (EAGLE design)
At the start: 80 x 126 mm, 78 parts, among them U1 CHG-4056, U2 FEATHER_WING_OLED

Commit message: edit enter
Parts:
- removed U$1: (no value), picoKey:STABILIZER
- added D4: 1N4148WS123, SamacSys_Parts:SOD-123
- added LED20: SK6812MINI-EH, picoKey:SK6812MINIE-H
- added S4: CPG135001D02V2, picoKey:KAILH_CHOC_V2
- moved TP1 14.5 mm to (71.5, 18.6)
- moved LED16 9.50 mm to (68.5, 35.2)
- moved D8 9.50 mm to (61.0, 24.6)
- moved S8 9.50 mm to (68.5, 24.6)
Connections:
- new net N$38: LED20.2, TP1.TP
- new net N$8: D4.A, S4.2
- net COL4: now also S4.1
- net GND: now also LED20.3
- net LED20: now also LED20.4; no longer TP1.TP
- net ROW1: now also D4.K
- net VSYS: now also LED20.1
Routing:
- net VSYS: track 589.5 -> 614.1 mm
- net COL4: track 113.7 -> 134.7 mm
- net LED20: track 5.28 -> 15.1 mm
- net LED17: track 100.3 -> 92.2 mm
- net ROW2: track 108.5 -> 100.8 mm, vias 2 -> 1
- net LED16: track 20.9 -> 14.9 mm
- net ROW1: track 110.4 -> 116.0 mm
- net N$8: track 0.00 -> 2.71 mm
- net N$38: track 0.00 -> 1.75 mm
- net GND: track 24.8 -> 26.0 mm, vias 70 -> 71
Other:
- board text added: "エンター スタビライザー"
