File: picoKey_230407.sch (EAGLE design)
At the start: 77 parts, among them U1 CHG-4056, U2 FEATHER_WING_OLED

Commit message: edit enter
Parts:
- added D4: 1N4148WS123, SamacSys_Parts:1N4148WS123
- added LED20: SK6812MINI-EH, picoKey:SK6812MINI-EH
- added S4: CPG135001D02V2, picoKey:CPG135001D02V2
Connections:
- new net N$38: LED20.DOUT, TP1.TP
- new net N$8: D4.A, S4.2
- net COL4: now also S4.1
- net GND: now also LED20.GND
- net LED20: now also LED20.DIN; no longer TP1.TP
- net ROW1: now also D4.K
- net VSYS: now also LED20.VDD
Other:
- moved on the sheet: TP1
Changed lines of the file:
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@@
 <part name="S2" library="picoKey" deviceset="CPG135001D02" device="V2" value="CPG135001D02V2"/>
 <part name="S3" library="picoKey" deviceset="CPG135001D02" device="V2" value="CPG135001D02V2"/>
+<part name="S4" library="picoKey" deviceset="CPG135001D02" device="V2" value="CPG135001D02V2"/>
 <part name="S5" library="picoKey" deviceset="CPG135001D02" device="V2" value="CPG135001D02V2"/>
 <part name="S6" library="picoKey" deviceset="CPG135001D02" device="V2" value="CPG135001D02V2"/>
@@
 <part name="D2" library="SamacSys_Parts" deviceset="1N4148WS" device="123" value="1N4148WS123"/>
 <part name="D3" library="SamacSys_Parts" deviceset="1N4148WS" device="123" value="1N4148WS123"/>
+<part name="D4" library="SamacSys_Parts" deviceset="1N4148WS" device="123" value="1N4148WS123"/>
 <part name="D5" library="SamacSys_Parts" deviceset="1N4148WS" device="123" value="1N4148WS123"/>
 <part name="D6" library="SamacSys_Parts" deviceset="1N4148WS" device="123" value="1N4148WS123"/>
@@
 <part name="LED19" library="picoKey" deviceset="SK6812MINI-E" device="H" value="SK6812MINI-EH"/>
 <part name="GND25" library="Miya_Supply" deviceset="G" device=""/>
+<part name="LED20" library="picoKey" deviceset="SK6812MINI-E" device="H" value="SK6812MINI-EH"/>
 <part name="TP1" library="testpad" library_urn="urn:adsk.eagle:library:385" deviceset="TP" device="TP06R" package3d_urn="urn:adsk.eagle:package:27954/1"/>
 <part name="TP2" library="testpad" library_urn="urn:adsk.eagle:library:385" deviceset="TP" device="TP06R" package3d_urn="urn:adsk.eagle:package:27954/1"/>
@@
 <attribute name="VALUE" x="101.6" y="142.24" size="1.778" layer="96" align="center-left"/>
 </instance>
+<instance part="S4" gate="G$1" x="137.16" y="146.05" smashed="yes">
+<attribute name="NAME" x="132.08" y="149.86" size="1.778" layer="95" align="center-left"/>
+<attribute name="VALUE" x="127" y="142.24" size="1.778" layer="96" align="center-left"/>
+</instance>
 <instance part="S5" gate="G$1" x="57.15" y="166.37" smashed="yes">
 <attribute name="NAME" x="52.07" y="170.18" size="1.778" layer="95" align="center-left"/>
@@
 <attribute name="NAME" x="115.57" y="134.62" size="1.778" layer="95" rot="R90" align="center-left"/>
 <attribute name="VALUE" x="123.19" y="134.62" size="1.778" layer="96" rot="R90" align="center-left"/>
+</instance>
+<instance part="D4" gate="G$1" x="146.05" y="138.43" smashed="yes" rot="R90">
+<attribute name="NAME" x="140.97" y="134.62" size="1.778" layer="95" rot="R90" align="center-left"/>
+<attribute name="VALUE" x="148.59" y="134.62" size="1.778" layer="96" rot="R90" align="center-left"/>
 </instance>
 <instance part="D5" gate="G$1" x="66.04" y="158.75" smashed="yes" rot="R90">
@@
 </instance>
 <instance part="GND25" gate="G$1" x="237.49" y="100.33" smashed="yes"/>
-<instance part="TP1" gate="G$1" x="233.68" y="115.57" smashed="yes">
-<attribute name="NAME" x="232.41" y="116.84" size="1.778" layer="95"/>
-<attribute name="TP_SIGNAL_NAME" x="234.95" y="114.3" size="1.778" layer="97"/>
+<instance part="LED20" gate="G$1" x="222.25" y="111.76" smashed="yes">
+<attribute name="NAME" x="213.36" y="116.84" size="1.778" layer="95" align="center-left"/>
+<attribute name="VALUE" x="213.36" y="106.68" size="1.778" layer="96" align="center-left"/>
+</instance>
+<instance part="TP1" gate="G$1" x="203.2" y="113.03" smashed="yes">
+<attribute name="NAME" x="201.93" y="114.3" size="1.778" layer="95"/>
+<attribute name="TP_SIGNAL_NAME" x="204.47" y="111.76" size="1.778" layer="97"/>
 </instance>
 <instance part="TP2" gate="G$1" x="88.9" y="58.42" smashed="yes" rot="R270">
@@
 <label x="125.73" y="233.68" size="1.778" layer="95" rot="R90" xref="yes"/>
 <wire x1="125.73" y1="144.78" x2="125.73" y2="165.1" width="0.1524" layer="91"/>
+<pinref part="S4" gate="G$1" pin="1"/>
 <wire x1="125.73" y1="165.1" x2="125.73" y2="185.42" width="0.1524" layer="91"/>
 <wire x1="125.73" y1="185.42" x2="125.73" y2="205.74" width="0.1524" layer="91"/>
@@
 <wire x1="120.65" y1="132.08" x2="146.05" y2="132.08" width="0.1524" layer="91"/>
 <junction x="120.65" y="132.08"/>
+<pinref part="D4" gate="G$1" pin="K"/>
 <wire x1="146.05" y1="132.08" x2="146.05" y2="134.62" width="0.1524" layer="91"/>
 </segment>
@@
 <net name="N$8" class="0">
 <segment>
+<pinref part="D4" gate="G$1" pin="A"/>
 <wire x1="146.05" y1="142.24" x2="146.05" y2="144.78" width="0.1524" layer="91"/>
+<pinref part="S4" gate="G$1" pin="2"/>
 <wire x1="143.51" y1="144.78" x2="146.05" y2="144.78" width="0.1524" layer="91"/>
 </segment>
@@
 </segment>
 <segment>
+<pinref part="LED20" gate="G$1" pin="VDD"/>
 <wire x1="210.82" y1="113.03" x2="207.01" y2="113.03" width="0.1524" layer="91"/>
 <wire x1="207.01" y1="113.03" x2="207.01" y2="120.65" width="0.1524" layer="91"/>
@@
 </segment>
 <segment>
+<pinref part="LED20" gate="G$1" pin="GND"/>
 <wire x1="233.68" y1="110.49" x2="237.49" y2="110.49" width="0.1524" layer="91"/>
 <pinref part="GND25" gate="G$1" pin="GND"/>
@@
 <wire x1="247.65" y1="110.49" x2="240.03" y2="110.49" width="0.1524" layer="91"/>
 <wire x1="240.03" y1="110.49" x2="240.03" y2="113.03" width="0.1524" layer="91"/>
+<pinref part="LED20" gate="G$1" pin="DIN"/>
 <wire x1="233.68" y1="113.03" x2="240.03" y2="113.03" width="0.1524" layer="91"/>
 <label x="238.76" y="113.03" size="1.778" layer="95"/>
-<pinref part="TP1" gate="G$1" pin="TP"/>
 </segment>
 </net>
@@
 </segment>
 </net>
+<net name="N$38" class="0">
+<segment>
+<pinref part="LED20" gate="G$1" pin="DOUT"/>
+<wire x1="210.82" y1="110.49" x2="203.2" y2="110.49" width="0.1524" layer="91"/>
+<pinref part="TP1" gate="G$1" pin="TP"/>
+</segment>
+</net>
