File: nrfKey_2401.brd (EAGLE design)
At the start: 80 x 126 mm, 78 parts, among them U1 CHG-4056, U2 FEATHER_WING_OLED

Commit message: add code
Parts:
- added C1: 1u, Miya_IC:C0603
- added C2: 0.1u, Miya_IC:C0603
- added IC1: TCK107AF,LF, SamacSys_Parts:SMV_1
- added R10: ND, Miya_IC:R0603
- added R11: 51, Miya_IC:R0603
- added U3: PIEZO_SOUNDER, my_lib:DINAMIC-SPK
- added U4: AE-NRF52840, picoKey:AE-NRF52840
- D21: value 1N4148WS -> RBE2VAM20ATR
- Q2: value (none) -> 2N7002
- R1: value 100k -> ND
- R7, R8: value 100k -> 4.7k
- S8: value CPG135001D02-SS -> CPG135001D02-SV2_V; device picoKey:CPG135001D02-S -> picoKey:KAILH_CHOC_V2_V
- moved R8 1.10 mm to (28.5, 101.0), turned to 180 degrees
- moved D21 0.10 mm to (58.6, 119.6)
Connections:
- new net N$1: R10.2, U2.16
- new net N$3: IC1.3, R11.2
- new net N$4: R11.1
- new net RUN: R10.1, X1.RUN
- new net VLED: C2.2, IC1.1, LED1.1, LED10.1, LED11.1, LED12.1, LED13.1, LED14.1, LED15.1, LED16.1, LED17.1, LED18.1, LED19.1, LED2.1, LED3.1, LED4.1, LED5.1, LED6.1, LED7.1, LED8.1, LED9.1, R8.1
- net GND: now also C1.1, C2.1, IC1.2
- net VSYS: now also C1.2, IC1.5; no longer LED1.1, LED10.1, LED11.1, LED12.1, LED13.1, LED14.1, LED15.1, LED16.1, LED17.1, LED18.1, LED19.1, LED2.1, LED3.1, LED4.1, LED5.1, LED6.1, LED7.1, LED8.1, LED9.1, R8.1
Routing:
- net VLED: track 0.00 -> 536.8 mm, vias 0 -> 28
- net VSYS: track 572.5 -> 40.0 mm, vias 29 -> 2
- net RUN: track 0.00 -> 23.1 mm
- net N$1: track 0.00 -> 19.6 mm
- net 3V3: track 63.8 -> 64.9 mm
- net SDA: track 22.7 -> 23.7 mm
- net SCL: track 26.3 -> 27.3 mm
- net LED3: track 24.2 -> 23.6 mm
- net B_BTN: track 25.6 -> 26.1 mm
- net C_BTN: track 63.7 -> 64.3 mm
- net GND: vias 70 -> 72
