File: picoKey_23/picoKey_2304.sch (EAGLE design)
At the start: 77 parts, among them U1 CHG-4056, U2 FEATHER_WING_OLED

Commit message: add code
Parts:
- added C1: 1u, Miya_IC:C_0603
- added C2: 0.1u, Miya_IC:C_0603
- added IC1: TCK107AF,LF, SamacSys_Parts:TCK107AF,LF
- added R10: ND, Miya_IC:R_0603
- added R11: 51, Miya_IC:R_0603
- D21: value 1N4148WS -> RBE2VAM20ATR
- Q2: value (none) -> 2N7002
- R1: value 100k -> ND
- R7, R8: value 100k -> 4.7k
- S8: value CPG135001D02-SS -> CPG135001D02-SV2_V; device picoKey:CPG135001D02-SS -> picoKey:CPG135001D02-SV2_V
Connections:
- new net N$1: R10.2, U2.RST
- new net N$3: IC1.CONTROL, R11.2
- new net N$4: R11.1
- new net RUN: R10.1, X1.RUN
- new net VLED: C2.2, IC1.VOUT, LED1.VDD, LED10.VDD, LED11.VDD, LED12.VDD, LED13.VDD, LED14.VDD, LED15.VDD, LED16.VDD, LED17.VDD, LED18.VDD, LED19.VDD, LED2.VDD, LED3.VDD, LED4.VDD, LED5.VDD, LED6.VDD, LED7.VDD, LED8.VDD, LED9.VDD, R8.1
- net GND: now also C1.1, C2.1, IC1.GND
- net VSYS: now also C1.2, IC1.VIN; no longer LED1.VDD, LED10.VDD, LED11.VDD, LED12.VDD, LED13.VDD, LED14.VDD, LED15.VDD, LED16.VDD, LED17.VDD, LED18.VDD, LED19.VDD, LED2.VDD, LED3.VDD, LED4.VDD, LED5.VDD, LED6.VDD, LED7.VDD, LED8.VDD, LED9.VDD, R8.1
Other:
- note added: "100k -> 10k?"
- note added: "4.7k->1.8k"
- note added: "R1はプルアップだとONにならない。"
- note added: "SK6812MINI 静止電流：1mA LED電源にロードスイッチ必要"
- note added: "ロードスイッチでもよかった TCK107AFLF"
- moved on the sheet: D21, Q1, R3, R4, U1
